Commit message: drifts are computed through tf trees

File: cartographer_ros/urdf/cinderella.urdf (robot description, URDF)
Before this commit: robot cinderella_3d, 4 links, 3 joints
Links:
- removed link laser_frame
- added link laser_link; visual cylinder length=0.07 radius=0.05
Joints:
- joint lidar_link_joint: child laser_frame -> laser_link

Commit message: add fake_gps to be published

File: cartographer_ros/urdf/cinderella.urdf (robot description, URDF)
Before this commit: robot cinderella_3d, 4 links, 3 joints
Joints:
- joint odom_link_joint: child odom_frame -> base_link; origin xyz=0.15 0. 0. rpy=0. 0. 0. -> xyz=-0.15 0. 0. rpy=0. 0. 0.; parent base_link -> odom_frame
